Commit message: Xacro added

File: workshop/workshop_description/urdf/car.xacro (robot description, xacro)
@@ -13,4 +13,6 @@
     <xacro:property name="h" value=".05"/>
     <xacro:property name="mass_wheel" value="0.2"/>
+    <!-- Including Color material for Gazebo -->
+    <xacro:include filename="$(find workshop_description)/urdf/materials.xacro"/>
     <link name="world"/>
     <joint name="fixed" type="fixed">
@@ -30,5 +32,4 @@
                 <box size="${length} ${width} ${height}"/>
             </geometry>
-            <material name="orange"/>
         </visual>
         <inertial>
@@ -41,5 +42,5 @@
     </link>
     <joint name="front_wheel_r_joint" type="continuous">
-        <origin xyz="${length/2} ${width/2} ${height/2}" rpy="0.0 0.0 0.0"/>
+        <origin xyz="${length/2} ${(h+width)/2} ${height/2}" rpy="0.0 0.0 0.0"/>
         <parent link="base_link"/>
         <child link="front_wheel_r_link"/>
@@ -48,5 +49,5 @@
     </joint>
     <joint name="front_wheel_l_joint" type="continuous">
-        <origin xyz="${length/2} ${-width/2} ${height/2}" rpy="0.0 0.0 0.0"/>
+        <origin xyz="${length/2} -${(h+width)/2} ${height/2}" rpy="0.0 0.0 0"/>
         <parent link="base_link"/>
         <child link="front_wheel_l_link"/>
@@ -55,14 +56,14 @@
     </joint>
     <joint name="back_wheel_r_joint" type="continuous">
-        <origin xyz="${length/2} ${width/2} ${height/2}" rpy="0.0 0.0 0.0"/>
+        <origin xyz="${-length/2} ${(h+width)/2} ${height/2}" rpy="0.0 0.0 0.0"/>
         <parent link="base_link"/>
-        <child link="front_wheel_r_link"/>
+        <child link="back_wheel_r_link"/>
         <axis xyz="0 1 0"/>
         <!-- <limit lower="0.0" upper="0.0" effort="0.0" velocity="0.0"/> -->
     </joint>
     <joint name="back_wheel_l_joint" type="continuous">
-        <origin xyz="${length/2} ${-width/2} ${height/2}" rpy="0.0 0.0 0.0"/>
+        <origin xyz="${-length/2} -${(h+width)/2} ${height/2}" rpy="0.0 0.0 0.0"/>
         <parent link="base_link"/>
-        <child link="front_wheel_l_link"/>
+        <child link="back_wheel_l_link"/>
         <axis xyz="0 1 0"/>
         <!-- <limit lower="0.0" upper="0.0" effort="0.0" velocity="0.0"/> -->

Commit message: Adding IMU

File: workshop/workshop_description/urdf/car.xacro (robot description, xacro)
@@ -15,9 +15,11 @@
     <!-- Including Color material for Gazebo -->
     <xacro:include filename="$(find workshop_description)/urdf/materials.xacro"/>
-    <link name="world"/>
-    <joint name="fixed" type="fixed">
-        <parent link="world"/>
-        <child link="base_link"/>
-    </joint>
+    <!--    Including sensors component-->
+    <xacro:include filename="$(find workshop_description)/urdf/component_snippets.xacro"/>
+<!--    <link name="world"/>-->
+<!--    <joint name="fixed" type="fixed">-->
+<!--        <parent link="world"/>-->
+<!--        <child link="base_link"/>-->
+<!--    </joint>-->
     <link name="base_link">
         <collision>
@@ -161,3 +163,74 @@
         </inertial>
     </link>
+    <joint name="imu_joint" type="fixed">
+        <origin xyz="0 0.0 ${height}" rpy="0.0 0.0 0.0"/>
+        <parent link="base_link"/>
+        <child link="imu_link"/>
+        <axis xyz="0.0 0.0 1.0"/>
+    </joint>
+    <link name="imu_link">
+    </link>
+    <!-- ADIS16448 IMU. -->
+    <xacro:imu_plugin_macro
+            namespace="${namespace}"
+            imu_suffix=""
+            parent_link="base_link"
+            imu_topic="imu"
+            mass_imu_sensor="0.00015"
+            gyroscope_noise_density="0.0003394"
+            gyroscope_random_walk="0.000038785"
+            gyroscope_bias_correlation_time="1000.0"
+            gyroscope_turn_on_bias_sigma="0.0087"
+            accelerometer_noise_density="0.004"
+            accelerometer_random_walk="0.006"
+            accelerometer_bias_correlation_time="300.0"
+            accelerometer_turn_on_bias_sigma="0.1960">
+        <inertia ixx="0.000001" ixy="0.0" ixz="0.0" iyy="0.000001" iyz="0.0" izz="0.000001"/>
+        <origin xyz="0 0 0" rpy="0 0 0"/>
+    </xacro:imu_plugin_macro>
+    <!-- Mount a Odometry Sensor -->
+    <!--    <xacro:odometry_plugin_macro-->
+    <!--            namespace="${namespace}"-->
+    <!--            odometry_sensor_suffix="1"-->
+    <!--            parent_link="${namespace}/base_link"-->
+    <!--            pose_topic="odometry_sensor/pose"-->
+    <!--            pose_with_covariance_topic="odometry_sensor/pose_with_covariance"-->
+    <!--            position_topic="odometry_sensor/position"-->
+    <!--            transform_topic="odometry_sensor/transform"-->
+    <!--            odometry_topic="odometry_sensor/odometry"-->
+    <!--            parent_frame_id="world"-->
+    <!--            child_frame_id="${namespace}/odometry_sensor1"-->
+    <!--            mass_odometry_sensor="0.00001"-->
+    <!--            measurement_divisor="1"-->
+    <!--            measurement_delay="0"-->
+    <!--            unknown_delay="0.0"-->
+    <!--            noise_normal_position="0 0 0"-->
+    <!--            noise_normal_quaternion="0 0 0"-->
+    <!--            noise_normal_linear_velocity="0 0 0"-->
+    <!--            noise_normal_angular_velocity="0 0 0"-->
+    <!--            noise_uniform_position=".0 0 0"-->
+    <!--            noise_uniform_quaternion="0 0 0"-->
+    <!--            noise_uniform_linear_velocity="0 0 0"-->
+    <!--            noise_uniform_angular_velocity="0 0 0"-->
+    <!--            enable_odometry_map="false"-->
+    <!--            odometry_map=""-->
+    <!--            image_scale="">-->
+    <!--        <inertia ixx="1e-10" ixy="0.0" ixz="0.0" iyy="1e-10" iyz="0.0" izz="1e-10" /> &lt;!&ndash; [kg m^2] [kg m^2] [kg m^2] [kg m^2] [kg m^2] [kg m^2] &ndash;&gt;-->
+    <!--        <origin xyz="0.0 0.0 0.0" rpy="0.0 0.0 0.0" />-->
+    <!--    </xacro:odometry_plugin_macro>-->
+    <!-- Mount a generic GPS sensor-->
+    <!--    <xacro:gps_plugin_macro-->
+    <!--            namespace="${namespace}"-->
+    <!--            gps_suffix=""-->
+    <!--            parent_link="${parent_link}"-->
+    <!--            gps_topic="gps"-->
+    <!--            ground_speed_topic="ground_speed"-->
+    <!--            mass_gps_sensor="0.015"-->
+    <!--            horizontal_pos_std_dev="3.0"-->
+    <!--            vertical_pos_std_dev="0.1"-->
+    <!--            horizontal_vel_std_dev="0.1"-->
+    <!--            vertical_vel_std_dev="0.1">-->
+    <!--        <inertia ixx="0.00001" ixy="0.0" ixz="0.0" iyy="0.00001" iyz="0.0" izz="0.00001" />-->
+    <!--        <origin xyz="0 0 0" rpy="0 0 0" />-->
+    <!--    </xacro:gps_plugin_macro>-->
 </robot>

Commit message: Finishing workshop1 URDF

File: workshop/workshop_description/urdf/car.xacro (robot description, xacro)
@@ -15,6 +15,4 @@
     <!-- Including Color material for Gazebo -->
     <xacro:include filename="$(find workshop_description)/urdf/materials.xacro"/>
-    <!--    Including sensors component-->
-    <xacro:include filename="$(find workshop_description)/urdf/component_snippets.xacro"/>
 <!--    <link name="world"/>-->
 <!--    <joint name="fixed" type="fixed">-->
@@ -163,74 +161,3 @@
         </inertial>
     </link>
-    <joint name="imu_joint" type="fixed">
-        <origin xyz="0 0.0 ${height}" rpy="0.0 0.0 0.0"/>
-        <parent link="base_link"/>
-        <child link="imu_link"/>
-        <axis xyz="0.0 0.0 1.0"/>
-    </joint>
-    <link name="imu_link">
-    </link>
-    <!-- ADIS16448 IMU. -->
-    <xacro:imu_plugin_macro
-            namespace="${namespace}"
-            imu_suffix=""
-            parent_link="base_link"
-            imu_topic="imu"
-            mass_imu_sensor="0.00015"
-            gyroscope_noise_density="0.0003394"
-            gyroscope_random_walk="0.000038785"
-            gyroscope_bias_correlation_time="1000.0"
-            gyroscope_turn_on_bias_sigma="0.0087"
-            accelerometer_noise_density="0.004"
-            accelerometer_random_walk="0.006"
-            accelerometer_bias_correlation_time="300.0"
-            accelerometer_turn_on_bias_sigma="0.1960">
-        <inertia ixx="0.000001" ixy="0.0" ixz="0.0" iyy="0.000001" iyz="0.0" izz="0.000001"/>
-        <origin xyz="0 0 0" rpy="0 0 0"/>
-    </xacro:imu_plugin_macro>
-    <!-- Mount a Odometry Sensor -->
-    <!--    <xacro:odometry_plugin_macro-->
-    <!--            namespace="${namespace}"-->
-    <!--            odometry_sensor_suffix="1"-->
-    <!--            parent_link="${namespace}/base_link"-->
-    <!--            pose_topic="odometry_sensor/pose"-->
-    <!--            pose_with_covariance_topic="odometry_sensor/pose_with_covariance"-->
-    <!--            position_topic="odometry_sensor/position"-->
-    <!--            transform_topic="odometry_sensor/transform"-->
-    <!--            odometry_topic="odometry_sensor/odometry"-->
-    <!--            parent_frame_id="world"-->
-    <!--            child_frame_id="${namespace}/odometry_sensor1"-->
-    <!--            mass_odometry_sensor="0.00001"-->
-    <!--            measurement_divisor="1"-->
-    <!--            measurement_delay="0"-->
-    <!--            unknown_delay="0.0"-->
-    <!--            noise_normal_position="0 0 0"-->
-    <!--            noise_normal_quaternion="0 0 0"-->
-    <!--            noise_normal_linear_velocity="0 0 0"-->
-    <!--            noise_normal_angular_velocity="0 0 0"-->
-    <!--            noise_uniform_position=".0 0 0"-->
-    <!--            noise_uniform_quaternion="0 0 0"-->
-    <!--            noise_uniform_linear_velocity="0 0 0"-->
-    <!--            noise_uniform_angular_velocity="0 0 0"-->
-    <!--            enable_odometry_map="false"-->
-    <!--            odometry_map=""-->
-    <!--            image_scale="">-->
-    <!--        <inertia ixx="1e-10" ixy="0.0" ixz="0.0" iyy="1e-10" iyz="0.0" izz="1e-10" /> &lt;!&ndash; [kg m^2] [kg m^2] [kg m^2] [kg m^2] [kg m^2] [kg m^2] &ndash;&gt;-->
-    <!--        <origin xyz="0.0 0.0 0.0" rpy="0.0 0.0 0.0" />-->
-    <!--    </xacro:odometry_plugin_macro>-->
-    <!-- Mount a generic GPS sensor-->
-    <!--    <xacro:gps_plugin_macro-->
-    <!--            namespace="${namespace}"-->
-    <!--            gps_suffix=""-->
-    <!--            parent_link="${parent_link}"-->
-    <!--            gps_topic="gps"-->
-    <!--            ground_speed_topic="ground_speed"-->
-    <!--            mass_gps_sensor="0.015"-->
-    <!--            horizontal_pos_std_dev="3.0"-->
-    <!--            vertical_pos_std_dev="0.1"-->
-    <!--            horizontal_vel_std_dev="0.1"-->
-    <!--            vertical_vel_std_dev="0.1">-->
-    <!--        <inertia ixx="0.00001" ixy="0.0" ixz="0.0" iyy="0.00001" iyz="0.0" izz="0.00001" />-->
-    <!--        <origin xyz="0 0 0" rpy="0 0 0" />-->
-    <!--    </xacro:gps_plugin_macro>-->
 </robot>
