Commit message: Adding sensor and actuator

File: workshop_description/urdf/car.xacro (robot description, xacro)
@@ -15,4 +15,6 @@
     <!-- Including Color material for Gazebo -->
     <xacro:include filename="$(find workshop_description)/urdf/materials.xacro"/>
+    <!--    Including sensors component-->
+    <xacro:include filename="$(find workshop_description)/urdf/component_snippets.xacro"/>
 <!--    <link name="world"/>-->
 <!--    <joint name="fixed" type="fixed">-->
@@ -161,3 +163,74 @@
         </inertial>
     </link>
+    <joint name="imu_joint" type="fixed">
+        <origin xyz="0 0.0 ${height}" rpy="0.0 0.0 0.0"/>
+        <parent link="base_link"/>
+        <child link="imu_link"/>
+        <axis xyz="0.0 0.0 1.0"/>
+    </joint>
+    <link name="imu_link">
+    </link>
+    <!-- ADIS16448 IMU. -->
+    <xacro:imu_plugin_macro
+            namespace="${namespace}"
+            imu_suffix=""
+            parent_link="base_link"
+            imu_topic="imu"
+            mass_imu_sensor="0.00015"
+            gyroscope_noise_density="0.0003394"
+            gyroscope_random_walk="0.000038785"
+            gyroscope_bias_correlation_time="1000.0"
+            gyroscope_turn_on_bias_sigma="0.0087"
+            accelerometer_noise_density="0.004"
+            accelerometer_random_walk="0.006"
+            accelerometer_bias_correlation_time="300.0"
+            accelerometer_turn_on_bias_sigma="0.1960">
+        <inertia ixx="0.000001" ixy="0.0" ixz="0.0" iyy="0.000001" iyz="0.0" izz="0.000001"/>
+        <origin xyz="0 0 0" rpy="0 0 0"/>
+    </xacro:imu_plugin_macro>
+    <!-- Mount a Odometry Sensor -->
+    <!--    <xacro:odometry_plugin_macro-->
+    <!--            namespace="${namespace}"-->
+    <!--            odometry_sensor_suffix="1"-->
+    <!--            parent_link="${namespace}/base_link"-->
+    <!--            pose_topic="odometry_sensor/pose"-->
+    <!--            pose_with_covariance_topic="odometry_sensor/pose_with_covariance"-->
+    <!--            position_topic="odometry_sensor/position"-->
+    <!--            transform_topic="odometry_sensor/transform"-->
+    <!--            odometry_topic="odometry_sensor/odometry"-->
+    <!--            parent_frame_id="world"-->
+    <!--            child_frame_id="${namespace}/odometry_sensor1"-->
+    <!--            mass_odometry_sensor="0.00001"-->
+    <!--            measurement_divisor="1"-->
+    <!--            measurement_delay="0"-->
+    <!--            unknown_delay="0.0"-->
+    <!--            noise_normal_position="0 0 0"-->
+    <!--            noise_normal_quaternion="0 0 0"-->
+    <!--            noise_normal_linear_velocity="0 0 0"-->
+    <!--            noise_normal_angular_velocity="0 0 0"-->
+    <!--            noise_uniform_position=".0 0 0"-->
+    <!--            noise_uniform_quaternion="0 0 0"-->
+    <!--            noise_uniform_linear_velocity="0 0 0"-->
+    <!--            noise_uniform_angular_velocity="0 0 0"-->
+    <!--            enable_odometry_map="false"-->
+    <!--            odometry_map=""-->
+    <!--            image_scale="">-->
+    <!--        <inertia ixx="1e-10" ixy="0.0" ixz="0.0" iyy="1e-10" iyz="0.0" izz="1e-10" /> &lt;!&ndash; [kg m^2] [kg m^2] [kg m^2] [kg m^2] [kg m^2] [kg m^2] &ndash;&gt;-->
+    <!--        <origin xyz="0.0 0.0 0.0" rpy="0.0 0.0 0.0" />-->
+    <!--    </xacro:odometry_plugin_macro>-->
+    <!-- Mount a generic GPS sensor-->
+    <!--    <xacro:gps_plugin_macro-->
+    <!--            namespace="${namespace}"-->
+    <!--            gps_suffix=""-->
+    <!--            parent_link="${parent_link}"-->
+    <!--            gps_topic="gps"-->
+    <!--            ground_speed_topic="ground_speed"-->
+    <!--            mass_gps_sensor="0.015"-->
+    <!--            horizontal_pos_std_dev="3.0"-->
+    <!--            vertical_pos_std_dev="0.1"-->
+    <!--            horizontal_vel_std_dev="0.1"-->
+    <!--            vertical_vel_std_dev="0.1">-->
+    <!--        <inertia ixx="0.00001" ixy="0.0" ixz="0.0" iyy="0.00001" iyz="0.0" izz="0.00001" />-->
+    <!--        <origin xyz="0 0 0" rpy="0 0 0" />-->
+    <!--    </xacro:gps_plugin_macro>-->
 </robot>

Commit message: Adding skin to URDF car

File: workshop_description/urdf/car.xacro (robot description, xacro)
@@ -4,12 +4,13 @@
     <xacro:property name="namespace" value="car"/>
     <xacro:property name="PI" value="3.1415926535897931"/>
+    <xacro:property name="skin_car" value="package://workshop_description/meshes/car/car.dae"/>
     <!-- Properties of base -->
     <xacro:property name="height" value=".2"/>
     <xacro:property name="width" value="1.2"/>
-    <xacro:property name="length" value="2"/>
+    <xacro:property name="length" value="2.5"/>
     <xacro:property name="mass_base" value="1"/>
     <!-- Properties of wheels    -->
-    <xacro:property name="radius" value="0.3"/>
-    <xacro:property name="h" value=".05"/>
+    <xacro:property name="radius" value="0.25"/>
+    <xacro:property name="h" value="0.05"/>
     <xacro:property name="mass_wheel" value="0.2"/>
     <!-- Including Color material for Gazebo -->
@@ -30,7 +31,7 @@
         </collision>
         <visual>
-            <origin xyz="0 0 ${height/2}" rpy="0 0 0"/>
-            <geometry>
-                <box size="${length} ${width} ${height}"/>
+            <origin xyz="0 0 -${height/2}" rpy="0 0 ${PI/2}"/>
+            <geometry>
+                <mesh filename="${skin_car}" scale="1 1 1"/>
             </geometry>
         </visual>

Commit message: Adding joint velocity control

File: workshop_description/urdf/car.xacro (robot description, xacro)
@@ -4,23 +4,25 @@
     <xacro:property name="namespace" value="car"/>
     <xacro:property name="PI" value="3.1415926535897931"/>
-    <xacro:property name="skin_car" value="package://workshop_description/meshes/car/car.dae"/>
+    <xacro:property name="skin_car" value="package://workshop_description/meshes/car/BMW.dae"/>
     <!-- Properties of base -->
     <xacro:property name="height" value=".2"/>
     <xacro:property name="width" value="1.2"/>
     <xacro:property name="length" value="2.5"/>
-    <xacro:property name="mass_base" value="1"/>
+    <xacro:property name="mass_base" value="10"/>
     <!-- Properties of wheels    -->
     <xacro:property name="radius" value="0.25"/>
     <xacro:property name="h" value="0.05"/>
-    <xacro:property name="mass_wheel" value="0.2"/>
+    <xacro:property name="mass_wheel" value="2"/>
     <!-- Including Color material for Gazebo -->
     <xacro:include filename="$(find workshop_description)/urdf/materials.xacro"/>
     <!--    Including sensors component-->
     <xacro:include filename="$(find workshop_description)/urdf/component_snippets.xacro"/>
-<!--    <link name="world"/>-->
-<!--    <joint name="fixed" type="fixed">-->
-<!--        <parent link="world"/>-->
-<!--        <child link="base_link"/>-->
-<!--    </joint>-->
+    <!--    Include link to Gazebo structure-->
+    <xacro:include filename="$(find workshop_description)/urdf/car.gazebo"/>
+    <!--    <link name="world"/>-->
+    <!--    <joint name="fixed" type="fixed">-->
+    <!--        <parent link="world"/>-->
+    <!--        <child link="base_link"/>-->
+    <!--    </joint>-->
     <link name="base_link">
         <collision>
@@ -31,5 +33,5 @@
         </collision>
         <visual>
-            <origin xyz="0 0 -${height/2}" rpy="0 0 ${PI/2}"/>
+            <origin xyz="0 0 -${height/2}" rpy="${PI/2} 0 ${PI}"/>
             <geometry>
                 <mesh filename="${skin_car}" scale="1 1 1"/>
@@ -172,4 +174,44 @@
     <link name="imu_link">
     </link>
+    <transmission name="front_wheel_r_tran">
+        <type>transmission_interface/SimpleTransmission</type>
+        <joint name="front_wheel_r_joint">
+            <hardwareInterface>hardware_interface/EffortJointInterface</hardwareInterface>
+        </joint>
+        <actuator name="front_wheel_r_motor">
+            <hardwareInterface>hardware_interface/EffortJointInterface</hardwareInterface>
+            <mechanicalReduction>1</mechanicalReduction>
+        </actuator>
+    </transmission>
+    <transmission name="front_wheel_l_tran">
+        <type>transmission_interface/SimpleTransmission</type>
+        <joint name="front_wheel_l_joint">
+            <hardwareInterface>hardware_interface/EffortJointInterface</hardwareInterface>
+        </joint>
+        <actuator name="front_wheel_l_motor">
+            <hardwareInterface>hardware_interface/EffortJointInterface</hardwareInterface>
+            <mechanicalReduction>1</mechanicalReduction>
+        </actuator>
+    </transmission>
+    <transmission name="back_wheel_r_tran">
+        <type>transmission_interface/SimpleTransmission</type>
+        <joint name="back_wheel_r_joint">
+            <hardwareInterface>hardware_interface/EffortJointInterface</hardwareInterface>
+        </joint>
+        <actuator name="back_wheel_r_motor">
+            <hardwareInterface>hardware_interface/EffortJointInterface</hardwareInterface>
+            <mechanicalReduction>1</mechanicalReduction>
+        </actuator>
+    </transmission>
+    <transmission name="back_wheel_l_tran">
+        <type>transmission_interface/SimpleTransmission</type>
+        <joint name="back_wheel_l_joint">
+            <hardwareInterface>hardware_interface/EffortJointInterface</hardwareInterface>
+        </joint>
+        <actuator name="back_wheel_l_motor">
+            <hardwareInterface>hardware_interface/EffortJointInterface</hardwareInterface>
+            <mechanicalReduction>1</mechanicalReduction>
+        </actuator>
+    </transmission>
     <!-- ADIS16448 IMU. -->
     <xacro:imu_plugin_macro
